Commit message: modify i5 urdf

File: aubo_description/urdf/aubo_i5.urdf (robot description, URDF)
Before this commit: robot aubo_i5, 8 links, 7 joints
Links:
- link foreArm_Link: mass 2.27145669098343 -> 2.88
- link shoulder_Link: mass 1.57658348693929 -> 5.05
- link upperArm_Link: mass 4.04175782265494 -> 11.28
- link wrist1_Link: mass 0.500477539188764 -> 1.62
- link wrist2_Link: mass 0.500477539245988 -> 1.62
- link wrist3_Link: mass 0.158309554874285 -> 0.5
Joints:
- joint foreArm_joint: limit lower=-3.05 upper=3.05 effort=0 velocity=0 -> lower=-3.05 upper=3.05 effort=0 velocity=2.5964
- joint shoulder_joint: limit lower=-3.05 upper=3.05 effort=0 velocity=0 -> lower=-3.05 upper=3.05 effort=0 velocity=2.5964
- joint upperArm_joint: limit lower=-3.05 upper=3.05 effort=0 velocity=0 -> lower=-3.05 upper=3.05 effort=0 velocity=2.5964
- joint wrist1_joint: limit lower=-3.05 upper=3.05 effort=0 velocity=0 -> lower=-3.05 upper=3.05 effort=0 velocity=3.1105
- joint wrist2_joint: limit lower=-3.05 upper=3.05 effort=0 velocity=0 -> lower=-3.05 upper=3.05 effort=0 velocity=3.1105
- joint wrist3_joint: limit lower=-3.05 upper=3.05 effort=0 velocity=0 -> lower=-3.05 upper=3.05 effort=0 velocity=3.1105
